Commit message: Refactor simulation architecture and add experiment comparison pipeline

File: src/my_robot_pkg/urdf/simple_rover.urdf.xacro (robot description, xacro)
@@ -3,174 +3,27 @@
   name="simple_rover"
   xmlns:xacro="http://www.ros.org/wiki/xacro">
-  <!-- ==================== -->
-  <!-- Geometric parameters -->
-  <!-- ==================== -->
-  <xacro:property name="body_length" value="1.0"/>
-  <xacro:property name="body_width" value="0.6"/>
-  <xacro:property name="body_height" value="0.2"/>
-  <xacro:property name="wheel_radius" value="0.15"/>
-  <xacro:property name="wheel_width" value="0.08"/>
-  <xacro:property name="wheel_x" value="0.35"/>
-  <xacro:property name="wheel_y" value="0.34"/>
-  <xacro:property name="wheel_z" value="-0.10"/>
-  <xacro:property name="arm_base_radius" value="0.10"/>
-  <xacro:property name="arm_base_height" value="0.08"/>
-  <xacro:property name="arm_link_1_length" value="0.40"/>
-  <xacro:property name="arm_link_2_length" value="0.36"/>
-  <!-- ========= -->
-  <!-- Materials -->
-  <!-- ========= -->
-  <material name="blue">
-    <color rgba="0.2 0.4 0.8 1.0"/>
-  </material>
-  <material name="black">
-    <color rgba="0.05 0.05 0.05 1.0"/>
-  </material>
-  <material name="gray">
-    <color rgba="0.4 0.4 0.4 1.0"/>
-  </material>
-  <material name="orange">
-    <color rgba="0.9 0.4 0.1 1.0"/>
-  </material>
-  <material name="yellow">
-    <color rgba="0.9 0.8 0.1 1.0"/>
-  </material>
-  <!-- =========== -->
-  <!-- Wheel macro -->
-  <!-- =========== -->
-  <xacro:macro name="wheel" params="name x y">
-    <link name="${name}">
-      <visual>
-        <geometry>
-          <cylinder
-            radius="${wheel_radius}"
-            length="${wheel_width}"/>
-        </geometry>
-        <material name="black"/>
-      </visual>
-    </link>
-    <joint name="${name}_joint" type="fixed">
-      <parent link="base_link"/>
-      <child link="${name}"/>
-      <origin
-        xyz="${x} ${y} ${wheel_z}"
-        rpy="1.5708 0 0"/>
-    </joint>
-  </xacro:macro>
-  <!-- =========== -->
-  <!-- Rover body  -->
-  <!-- =========== -->
-  <link name="base_link">
-    <visual>
-      <geometry>
-        <box size="${body_length} ${body_width} ${body_height}"/>
-      </geometry>
-      <material name="blue"/>
-    </visual>
-  </link>
-  <!-- Wheels created from one reusable macro -->
-  <xacro:wheel
-    name="front_left_wheel"
-    x="${wheel_x}"
-    y="${wheel_y}"/>
-  <xacro:wheel
-    name="front_right_wheel"
-    x="${wheel_x}"
-    y="${-wheel_y}"/>
-  <xacro:wheel
-    name="rear_left_wheel"
-    x="${-wheel_x}"
-    y="${wheel_y}"/>
-  <xacro:wheel
-    name="rear_right_wheel"
-    x="${-wheel_x}"
-    y="${-wheel_y}"/>
-  <!-- ======== -->
-  <!-- Arm base -->
-  <!-- ======== -->
-  <link name="arm_base">
-    <visual>
-      <geometry>
-        <cylinder
-          radius="${arm_base_radius}"
-          length="${arm_base_height}"/>
-      </geometry>
-      <material name="gray"/>
-    </visual>
-  </link>
-  <joint name="arm_base_joint" type="fixed">
-    <parent link="base_link"/>
-    <child link="arm_base"/>
-    <origin xyz="0 0 0.14" rpy="0 0 0"/>
-  </joint>
-  <!-- ========== -->
-  <!-- Arm link 1 -->
-  <!-- ========== -->
-  <link name="arm_link_1">
-    <visual>
-      <origin
-        xyz="0 0 ${arm_link_1_length / 2.0}"
-        rpy="0 0 0"/>
-      <geometry>
-        <box size="0.08 0.08 ${arm_link_1_length}"/>
-      </geometry>
-      <material name="orange"/>
-    </visual>
-  </link>
-  <joint name="shoulder_joint" type="revolute">
-    <parent link="arm_base"/>
-    <child link="arm_link_1"/>
-    <origin xyz="0 0 0.04" rpy="0 0 0"/>
-    <axis xyz="0 1 0"/>
-    <limit
-      lower="-1.57"
-      upper="1.57"
-      effort="20"
-      velocity="1.0"/>
-  </joint>
-  <!-- ========== -->
-  <!-- Arm link 2 -->
-  <!-- ========== -->
-  <link name="arm_link_2">
-    <visual>
-      <origin
-        xyz="0 0 ${arm_link_2_length / 2.0}"
-        rpy="0 0 0"/>
-      <geometry>
-        <box size="0.07 0.07 ${arm_link_2_length}"/>
-      </geometry>
-      <material name="yellow"/>
-    </visual>
-  </link>
-  <joint name="elbow_joint" type="revolute">
-    <parent link="arm_link_1"/>
-    <child link="arm_link_2"/>
-    <origin
-      xyz="0 0 ${arm_link_1_length}"
-      rpy="0 0 0"/>
-    <axis xyz="0 1 0"/>
-    <limit
-      lower="-1.57"
-      upper="1.57"
-      effort="20"
-      velocity="1.0"/>
-  </joint>
-  <!-- ====== -->
-  <!-- Camera -->
-  <!-- ====== -->
-  <link name="camera_link">
-    <visual>
-      <geometry>
-        <box size="0.14 0.10 0.08"/>
-      </geometry>
-      <material name="black"/>
-    </visual>
-  </link>
-  <joint name="camera_joint" type="fixed">
-    <parent link="arm_link_2"/>
-    <child link="camera_link"/>
-    <origin
-      xyz="0 0 ${arm_link_2_length + 0.04}"
-      rpy="0 0 0"/>
-  </joint>
+  <!-- =============================================== -->
+  <!-- Configuration                                   -->
+  <!-- =============================================== -->
+  <xacro:arg name="config_file" default=""/>
+  <xacro:property
+    name="config"
+    value="${xacro.load_yaml('$(arg config_file)')}"/>
+  <xacro:property
+    name="rover"
+    value="${config['rover']}"/>
+  <!-- =============================================== -->
+  <!-- Components                                      -->
+  <!-- =============================================== -->
+  <xacro:include filename="inertial_macros.xacro"/>
+  <xacro:include filename="rover_base.xacro"/>
+  <xacro:include filename="rover_arm.xacro"/>
+  <xacro:include filename="gazebo_plugins.xacro"/>
+  <xacro:include filename="materials.xacro"/>
+  <!-- =============================================== -->
+  <!-- Robot assembly                                  -->
+  <!-- =============================================== -->
+  <xacro:rover_base rover="${rover}"/>
+  <xacro:rover_arm rover="${rover}"/>
+  <xacro:gazebo_plugins rover="${rover}"/>
 </robot>
