Commit message: refactor robot models with generic arm kinematics and shared robot parameters

File: src/robot_description/urdf/robot_arm.xacro (robot description, xacro)
@@ -71,4 +71,17 @@
       name="camera_mass"
       value="${robot['arm']['camera']['mass']}"/>
+    <!-- Joints -->
+    <xacro:property
+      name="base_yaw_joint_cfg"
+      value="${robot['arm']['joints']['base_yaw']}"/>
+    <xacro:property
+      name="shoulder_joint_cfg"
+      value="${robot['arm']['joints']['shoulder']}"/>
+    <xacro:property
+      name="elbow_joint_cfg"
+      value="${robot['arm']['joints']['elbow']}"/>
+    <xacro:property
+      name="wrist_joint_cfg"
+      value="${robot['arm']['joints']['wrist']}"/>
     <!-- ============================================= -->
     <!-- Arm base                                      -->
@@ -101,12 +114,15 @@
         xyz="0 0 ${body_height / 2.0 + arm_base_height / 2.0}"
         rpy="0 0 0"/>
-      <axis xyz="0 0 1"/>
+      <axis
+        xyz="${base_yaw_joint_cfg['axis'][0]}
+             ${base_yaw_joint_cfg['axis'][1]}
+             ${base_yaw_joint_cfg['axis'][2]}"/>
       <limit
-        lower="-3.14"
-        upper="3.14"
-        effort="20"
-        velocity="1.0"/>
+        lower="${base_yaw_joint_cfg['lower']}"
+        upper="${base_yaw_joint_cfg['upper']}"
+        effort="${base_yaw_joint_cfg['effort']}"
+        velocity="${base_yaw_joint_cfg['velocity']}"/>
       <dynamics
-        damping="0.1"
+        damping="${base_yaw_joint_cfg['damping']}"
         friction="0.0"/>
     </joint>
@@ -151,12 +167,15 @@
         xyz="0 0 ${arm_base_height / 2.0}"
         rpy="0 0 0"/>
-      <axis xyz="0 -1 0"/>
+      <axis
+        xyz="${shoulder_joint_cfg['axis'][0]}
+             ${shoulder_joint_cfg['axis'][1]}
+             ${shoulder_joint_cfg['axis'][2]}"/>
       <limit
-        lower="-1.57"
-        upper="1.57"
-        effort="20"
-        velocity="1.0"/>
+        lower="${shoulder_joint_cfg['lower']}"
+        upper="${shoulder_joint_cfg['upper']}"
+        effort="${shoulder_joint_cfg['effort']}"
+        velocity="${shoulder_joint_cfg['velocity']}"/>
       <dynamics
-        damping="0.2"
+        damping="${shoulder_joint_cfg['damping']}"
         friction="0.0"/>
     </joint>
@@ -201,12 +220,15 @@
         xyz="${arm_link_1_length} 0 0"
         rpy="0 0 0"/>
-      <axis xyz="0 -1 0"/>
+      <axis
+        xyz="${elbow_joint_cfg['axis'][0]}
+             ${elbow_joint_cfg['axis'][1]}
+             ${elbow_joint_cfg['axis'][2]}"/>
       <limit
-        lower="-1.57"
-        upper="1.57"
-        effort="20"
-        velocity="1.0"/>
+        lower="${elbow_joint_cfg['lower']}"
+        upper="${elbow_joint_cfg['upper']}"
+        effort="${elbow_joint_cfg['effort']}"
+        velocity="${elbow_joint_cfg['velocity']}"/>
       <dynamics
-        damping="0.2"
+        damping="${elbow_joint_cfg['damping']}"
         friction="0.0"/>
     </joint>
@@ -251,12 +273,15 @@
         xyz="${arm_link_2_length} 0 0"
         rpy="0 0 0"/>
-      <axis xyz="0 -1 0"/>
+      <axis
+        xyz="${wrist_joint_cfg['axis'][0]}
+             ${wrist_joint_cfg['axis'][1]}
+             ${wrist_joint_cfg['axis'][2]}"/>
       <limit
-        lower="-1.57"
-        upper="1.57"
-        effort="10"
-        velocity="1.5"/>
+        lower="${wrist_joint_cfg['lower']}"
+        upper="${wrist_joint_cfg['upper']}"
+        effort="${wrist_joint_cfg['effort']}"
+        velocity="${wrist_joint_cfg['velocity']}"/>
       <dynamics
-        damping="0.15"
+        damping="${wrist_joint_cfg['damping']}"
         friction="0.0"/>
     </joint>

Commit message: Complete robot models v1 and optical camera integration

File: src/robot_description/urdf/robot_arm.xacro (robot description, xacro)
@@ -320,4 +320,19 @@
         rpy="0 0 0"/>
     </joint>
+    <!-- ============================================= -->
+    <!-- Camera optical frame                          -->
+    <!-- ROS optical convention:                       -->
+    <!--   x -> right                                  -->
+    <!--   y -> down                                   -->
+    <!--   z -> forward                                -->
+    <!-- ============================================= -->
+    <link name="camera_optical_frame"/>
+    <joint name="camera_optical_joint" type="fixed">
+      <parent link="camera_link"/>
+      <child link="camera_optical_frame"/>
+      <origin
+        xyz="0 0 0"
+        rpy="-1.57079632679 0 -1.57079632679"/>
+    </joint>
   </xacro:macro>
 </robot>
